File: hardware/mainpanel/mainpanel.brd (EAGLE design)
At the start: 80 x 80 mm, 2 parts

Commit message: Add components to sch
Parts:
- added B3: (no value), Frcy:UPUTRONICS-UBLOX-PICO
- added B4: (no value), Frcy:SPARKFUN-OPENLOG
- B1: value NUCLEO-32 -> (none)
Connections:
- new net CDH-RX: B1.D0/RX
- new net CDH-TX: B1.D1/TX
- new net GPS-SCL: B1.D5, B3.SCL
- new net GPS-SDA: B1.D4, B3.SDA
- new net GRN: B4.GRN
- new net LOG-UART: B1.A7, B4.RXI
- new net SPI-CS-ADC: B1.D6
- new net SPI-CS-ENV: B1.D3
- new net SPI-MISO: B1.A5
- new net SPI-MOSI: B1.D2
- new net SPI-SCK: B1.A1
- new net TEMP-OW: B1.D9
- net GND: now also B3.GND, B4.GND
- net VCC: now also B3.VCC, B4.VCC
Changed lines of the file:
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@@
 </autorouter>
 <elements>
-<element name="B1" library="Frcy" package="NUCLEO-32" value="NUCLEO-32" x="49.4" y="36.86" rot="R270"/>
+<element name="B1" library="Frcy" package="NUCLEO-32" value="" x="49.4" y="36.86" rot="R270"/>
 <element name="B2" library="Frcy" package="BOSCH-BNO055" value="BOSCH-BNO055" x="61.67" y="15.77" rot="R180"/>
+<element name="B3" library="Frcy" package="UPUTRONICS-UBLOX-PICO" value="" x="-22" y="6"/>
+<element name="B4" library="Frcy" package="SPARKFUN-OPENLOG" value="" x="-14" y="-11"/>
 </elements>
 <signals>
@@
 <contactref element="B1" pad="VIN"/>
 <contactref element="B2" pad="VIN"/>
+<contactref element="B3" pad="VCC"/>
+<contactref element="B4" pad="VCC"/>
 <wire x1="68.02" y1="24.66" x2="65.91" y2="29.24" width="0" layer="19" extent="1-1"/>
+<wire x1="-8.03" y1="7.27" x2="65.91" y2="29.24" width="0" layer="19" extent="1-1"/>
+<wire x1="-12.73" y1="-19.128" x2="-8.03" y2="7.27" width="0" layer="19" extent="1-1"/>
 </signal>
 <signal name="GND">
@@
 <vertex x="0" y="0"/>
 </polygon>
+<contactref element="B3" pad="GND"/>
+<contactref element="B4" pad="GND"/>
+<wire x1="63.37" y1="29.24" x2="58.29" y2="44.48" width="0" layer="19" extent="1-1"/>
+<wire x1="62.94" y1="24.66" x2="63.37" y2="29.24" width="0" layer="19" extent="1-1"/>
+<wire x1="-10.57" y1="7.27" x2="62.94" y2="24.66" width="0" layer="19" extent="1-1"/>
+<wire x1="-10.19" y1="-19.128" x2="-10.57" y2="7.27" width="0" layer="19" extent="1-1"/>
 </signal>
 <signal name="IMU-SDA">
@@
 <wire x1="53.21" y1="29.24" x2="57.86" y2="24.66" width="0" layer="19" extent="1-1"/>
 </signal>
+<signal name="GRN">
+<contactref element="B4" pad="GRN"/>
+</signal>
+<signal name="GPS-SDA">
+<contactref element="B3" pad="SDA"/>
+<contactref element="B1" pad="D4"/>
+<wire x1="-20.73" y1="7.27" x2="50.67" y2="44.48" width="0" layer="19" extent="1-1"/>
+</signal>
+<signal name="GPS-SCL">
+<contactref element="B3" pad="SCL"/>
+<contactref element="B1" pad="D5"/>
+<wire x1="-18.19" y1="7.27" x2="48.13" y2="44.48" width="0" layer="19" extent="1-1"/>
+</signal>
+<signal name="LOG-UART">
+<contactref element="B4" pad="RXI"/>
+<contactref element="B1" pad="A7"/>
+<wire x1="-17.81" y1="-19.128" x2="55.75" y2="29.24" width="0" layer="19" extent="1-1"/>
+</signal>
+<signal name="CDH-TX">
+<contactref element="B1" pad="D1/TX"/>
+</signal>
+<signal name="CDH-RX">
+<contactref element="B1" pad="D0/RX"/>
+</signal>
+<signal name="SPI-MOSI">
+<contactref element="B1" pad="D2"/>
+</signal>
+<signal name="SPI-CS-ADC">
+<contactref element="B1" pad="D6"/>
+</signal>
+<signal name="TEMP-OW">
+<contactref element="B1" pad="D9"/>
+</signal>
+<signal name="SPI-SCK">
+<contactref element="B1" pad="A1"/>
+</signal>
+<signal name="SPI-MISO">
+<contactref element="B1" pad="A5"/>
+</signal>
+<signal name="SPI-CS-ENV">
+<contactref element="B1" pad="D3"/>
+</signal>
 </signals>

Commit message: Place components on brd
Parts:
- moved B3 90.4 mm to (58.0, 48.0)
- moved B4 84.4 mm to (66.0, 16.0), turned to 180 degrees
- moved B2 22.0 mm to (39.7, 15.8)
- moved B1 1.00 mm to (48.4, 36.9)
Changed lines of the file:
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@@
 </autorouter>
 <elements>
-<element name="B1" library="Frcy" package="NUCLEO-32" value="" x="49.4" y="36.86" rot="R270"/>
-<element name="B2" library="Frcy" package="BOSCH-BNO055" value="BOSCH-BNO055" x="61.67" y="15.77" rot="R180"/>
-<element name="B3" library="Frcy" package="UPUTRONICS-UBLOX-PICO" value="" x="-22" y="6"/>
-<element name="B4" library="Frcy" package="SPARKFUN-OPENLOG" value="" x="-14" y="-11"/>
+<element name="B1" library="Frcy" package="NUCLEO-32" value="" x="48.4" y="36.86" rot="R270"/>
+<element name="B2" library="Frcy" package="BOSCH-BNO055" value="BOSCH-BNO055" x="39.67" y="15.77" rot="R180"/>
+<element name="B3" library="Frcy" package="UPUTRONICS-UBLOX-PICO" value="" x="58" y="48"/>
+<element name="B4" library="Frcy" package="SPARKFUN-OPENLOG" value="" x="66" y="16" rot="R180"/>
 </elements>
 <signals>
@@
 <contactref element="B3" pad="VCC"/>
 <contactref element="B4" pad="VCC"/>
-<wire x1="68.02" y1="24.66" x2="65.91" y2="29.24" width="0" layer="19" extent="1-1"/>
-<wire x1="-8.03" y1="7.27" x2="65.91" y2="29.24" width="0" layer="19" extent="1-1"/>
-<wire x1="-12.73" y1="-19.128" x2="-8.03" y2="7.27" width="0" layer="19" extent="1-1"/>
+<wire x1="64.91" y1="29.24" x2="71.97" y2="49.27" width="0" layer="19" extent="1-1"/>
+<wire x1="64.73" y1="24.128" x2="64.91" y2="29.24" width="0" layer="19" extent="1-1"/>
+<wire x1="46.02" y1="24.66" x2="64.73" y2="24.128" width="0" layer="19" extent="1-1"/>
 </signal>
 <signal name="GND">
@@
 <contactref element="B3" pad="GND"/>
 <contactref element="B4" pad="GND"/>
-<wire x1="63.37" y1="29.24" x2="58.29" y2="44.48" width="0" layer="19" extent="1-1"/>
-<wire x1="62.94" y1="24.66" x2="63.37" y2="29.24" width="0" layer="19" extent="1-1"/>
-<wire x1="-10.57" y1="7.27" x2="62.94" y2="24.66" width="0" layer="19" extent="1-1"/>
-<wire x1="-10.19" y1="-19.128" x2="-10.57" y2="7.27" width="0" layer="19" extent="1-1"/>
 </signal>
 <signal name="IMU-SDA">
 <contactref element="B2" pad="SDA"/>
 <contactref element="B1" pad="D12"/>
-<wire x1="30.35" y1="44.48" x2="60.4" y2="24.66" width="0" layer="19" extent="1-1"/>
+<wire x1="38.4" y1="24.66" x2="29.35" y2="44.48" width="0" layer="19" extent="1-1"/>
 </signal>
 <signal name="IMU-SCL">
 <contactref element="B2" pad="SCL"/>
 <contactref element="B1" pad="A6"/>
-<wire x1="53.21" y1="29.24" x2="57.86" y2="24.66" width="0" layer="19" extent="1-1"/>
+<wire x1="35.86" y1="24.66" x2="52.21" y2="29.24" width="0" layer="19" extent="1-1"/>
 </signal>
 <signal name="GRN">
@@
 <contactref element="B3" pad="SDA"/>
 <contactref element="B1" pad="D4"/>
-<wire x1="-20.73" y1="7.27" x2="50.67" y2="44.48" width="0" layer="19" extent="1-1"/>
+<wire x1="49.67" y1="44.48" x2="59.27" y2="49.27" width="0" layer="19" extent="1-1"/>
 </signal>
 <signal name="GPS-SCL">
 <contactref element="B3" pad="SCL"/>
 <contactref element="B1" pad="D5"/>
-<wire x1="-18.19" y1="7.27" x2="48.13" y2="44.48" width="0" layer="19" extent="1-1"/>
+<wire x1="47.13" y1="44.48" x2="61.81" y2="49.27" width="0" layer="19" extent="1-1"/>
 </signal>
 <signal name="LOG-UART">
 <contactref element="B4" pad="RXI"/>
 <contactref element="B1" pad="A7"/>
-<wire x1="-17.81" y1="-19.128" x2="55.75" y2="29.24" width="0" layer="19" extent="1-1"/>
+<wire x1="54.75" y1="29.24" x2="69.81" y2="24.128" width="0" layer="19" extent="1-1"/>
 </signal>
 <signal name="CDH-TX">

Commit message: Add connectors
Parts:
- added J1, J2, J3: 90136-104, con-molex-c-grid:90136-1?04
- added J4: 90136-108, con-molex-c-grid:90136-1?08
Connections:
- new net N$1: J3.1
- new net N$10: J4.6
- new net N$11: J4.7
- new net N$12: J4.8
- new net N$2: J3.2
- new net N$3: J3.3
- new net N$4: J3.4
- new net N$5: J4.1
- new net N$6: J4.2
- new net N$7: J4.3
- new net N$8: J4.4
- new net N$9: J4.5
- net CDH-RX: now also J1.3
- net CDH-TX: now also J1.2
- net GND: now also J1.1, J2.1, J2.3
- net TEMP-OW: now also J2.2
- net VCC: now also J1.4, J2.4
Changed lines of the file:
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@@
 </variantdefs>
 <classes>
-<class number="0" name="default" width="0" drill="0">
+<class number="0" name="default" width="0.8128" drill="0.8">
+<clearance class="0" value="0.4064"/>
 </class>
 </classes>
@@
 <param name="RoutingGrid" value="50mil"/>
 <param name="AutoGrid" value="1"/>
-<param name="Efforts" value="0"/>
+<param name="Efforts" value="1"/>
 <param name="TopRouterVariant" value="1"/>
 <param name="tpViaShape" value="round"/>
@@
 <element name="B3" library="Frcy" package="UPUTRONICS-UBLOX-PICO" value="" x="58" y="48"/>
 <element name="B4" library="Frcy" package="SPARKFUN-OPENLOG" value="" x="66" y="16" rot="R180"/>
+<element name="J1" library="con-molex-c-grid" package="90136-1?04" value="90136-104" x="46" y="72"/>
+<element name="J2" library="con-molex-c-grid" package="90136-1?04" value="90136-104" x="29" y="72"/>
+<element name="J3" library="con-molex-c-grid" package="90136-1?04" value="90136-104" x="12" y="41" rot="R90"/>
+<element name="J4" library="con-molex-c-grid" package="90136-1?08" value="90136-108" x="12" y="19" rot="R90"/>
 </elements>
 <signals>
@@
 <contactref element="B3" pad="VCC"/>
 <contactref element="B4" pad="VCC"/>
+<contactref element="J1" pad="4"/>
+<contactref element="J2" pad="4"/>
 <wire x1="64.91" y1="29.24" x2="71.97" y2="49.27" width="0" layer="19" extent="1-1"/>
 <wire x1="64.73" y1="24.128" x2="64.91" y2="29.24" width="0" layer="19" extent="1-1"/>
 <wire x1="46.02" y1="24.66" x2="64.73" y2="24.128" width="0" layer="19" extent="1-1"/>
+<wire x1="49.81" y1="72" x2="71.97" y2="49.27" width="0" layer="19" extent="1-1"/>
+<wire x1="32.81" y1="72" x2="49.81" y2="72" width="0" layer="19" extent="1-1"/>
 </signal>
 <signal name="GND">
@@
 <contactref element="B3" pad="GND"/>
 <contactref element="B4" pad="GND"/>
+<contactref element="J1" pad="1"/>
+<contactref element="J2" pad="1"/>
+<contactref element="J2" pad="3"/>
 </signal>
 <signal name="IMU-SDA">
@@
 <signal name="CDH-TX">
 <contactref element="B1" pad="D1/TX"/>
+<contactref element="J1" pad="2"/>
+<wire x1="64.91" y1="44.48" x2="44.73" y2="72" width="0" layer="19" extent="1-1"/>
 </signal>
 <signal name="CDH-RX">
 <contactref element="B1" pad="D0/RX"/>
+<contactref element="J1" pad="3"/>
+<wire x1="62.37" y1="44.48" x2="47.27" y2="72" width="0" layer="19" extent="1-1"/>
 </signal>
 <signal name="SPI-MOSI">
@@
 <signal name="TEMP-OW">
 <contactref element="B1" pad="D9"/>
+<contactref element="J2" pad="2"/>
+<wire x1="36.97" y1="44.48" x2="27.73" y2="72" width="0" layer="19" extent="1-1"/>
 </signal>
 <signal name="SPI-SCK">
@@
 <contactref element="B1" pad="D3"/>
 </signal>
+<signal name="N$1">
+<contactref element="J3" pad="1"/>
+</signal>
+<signal name="N$2">
+<contactref element="J3" pad="2"/>
+</signal>
+<signal name="N$3">
+<contactref element="J3" pad="3"/>
+</signal>
+<signal name="N$4">
+<contactref element="J3" pad="4"/>
+</signal>
+<signal name="N$5">
+<contactref element="J4" pad="1"/>
+</signal>
+<signal name="N$6">
+<contactref element="J4" pad="2"/>
+</signal>
+<signal name="N$7">
+<contactref element="J4" pad="3"/>
+</signal>
+<signal name="N$8">
+<contactref element="J4" pad="4"/>
+</signal>
+<signal name="N$9">
+<contactref element="J4" pad="5"/>
+</signal>
+<signal name="N$10">
+<contactref element="J4" pad="6"/>
+</signal>
+<signal name="N$11">
+<contactref element="J4" pad="7"/>
+</signal>
+<signal name="N$12">
+<contactref element="J4" pad="8"/>
+</signal>
 </signals>

Commit message: Add more connectors
Parts:
- added J5: 90136-104, con-molex-c-grid:90136-1?04
- J1: value 90136-104 -> 90136-106; device con-molex-c-grid:90136-1?04 -> con-molex-c-grid:90136-1?06
- moved J3 49.0 mm to (50.0, 72.0), turned to 0 degrees
- moved J1 31.0 mm to (15.0, 72.0)
- moved J4 9.22 mm to (10.0, 28.0)
- moved J2 5.00 mm to (34.0, 72.0)
- moved B1 1.00 mm to (47.4, 36.9)
Connections:
- removed net 3V3: B1.3V3
- removed net N$1: J3.1
- removed net N$10: J4.6
- removed net N$11: J4.7
- removed net N$12: J4.8
- removed net N$2: J3.2
- removed net N$3: J3.3
- removed net N$4: J3.4
- removed net N$5: J4.1
- removed net N$6: J4.2
- removed net N$7: J4.3
- removed net N$8: J4.4
- removed net N$9: J4.5
- removed net SPI-CS-ADC: B1.D6
- new net DBG-RX: B1.A2, J3.3
- new net DBG-TX: B1.A0, J3.4
- new net GPS-RX: B3.RXD, J3.1
- new net GPS-TX: B3.TXD, J3.2
- new net N$13: B1.RST@2
- new net SPI-CS-ADCS: B1.D6, J4.2
- new net SPI-CS-SUN: B1.D10, J4.3
- new net SUN-RX: B1.A4, J5.2
- new net SUN-TX: B1.A3, J5.3
- new net VIN: B1.VIN
- net CDH-RX: now also J1.4; no longer J1.3
- net CDH-TX: now also J1.3; no longer J1.2
- net GND: now also J1.5, J1.6, J4.5, J5.1
- net SPI-CS-ENV: now also J4.1
- net SPI-MISO: now also J4.6
- net SPI-MOSI: now also J4.7
- net SPI-SCK: now also J4.4
- net VCC: now also B1.3V3, J1.2, J4.8, J5.4; no longer B1.VIN, J1.4
Changed lines of the file:
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@@
 <autorouter>
 <pass name="Default">
-<param name="RoutingGrid" value="50mil"/>
+<param name="RoutingGrid" value="0.125mm"/>
 <param name="AutoGrid" value="1"/>
 <param name="Efforts" value="1"/>
 <param name="TopRouterVariant" value="1"/>
 <param name="tpViaShape" value="round"/>
-<param name="PrefDir.1" value="a"/>
+<param name="PrefDir.1" value="*"/>
 <param name="PrefDir.2" value="0"/>
 <param name="PrefDir.3" value="0"/>
@@
 <param name="PrefDir.14" value="0"/>
 <param name="PrefDir.15" value="0"/>
-<param name="PrefDir.16" value="a"/>
+<param name="PrefDir.16" value="*"/>
 <param name="cfVia" value="8"/>
 <param name="cfNonPref" value="5"/>
@@
 </autorouter>
 <elements>
-<element name="B1" library="Frcy" package="NUCLEO-32" value="" x="48.4" y="36.86" rot="R270"/>
+<element name="B1" library="Frcy" package="NUCLEO-32" value="" x="47.4" y="36.86" rot="R270"/>
 <element name="B2" library="Frcy" package="BOSCH-BNO055" value="BOSCH-BNO055" x="39.67" y="15.77" rot="R180"/>
 <element name="B3" library="Frcy" package="UPUTRONICS-UBLOX-PICO" value="" x="58" y="48"/>
 <element name="B4" library="Frcy" package="SPARKFUN-OPENLOG" value="" x="66" y="16" rot="R180"/>
-<element name="J1" library="con-molex-c-grid" package="90136-1?04" value="90136-104" x="46" y="72"/>
-<element name="J2" library="con-molex-c-grid" package="90136-1?04" value="90136-104" x="29" y="72"/>
-<element name="J3" library="con-molex-c-grid" package="90136-1?04" value="90136-104" x="12" y="41" rot="R90"/>
-<element name="J4" library="con-molex-c-grid" package="90136-1?08" value="90136-108" x="12" y="19" rot="R90"/>
+<element name="J2" library="con-molex-c-grid" package="90136-1?04" value="90136-104" x="34" y="72"/>
+<element name="J3" library="con-molex-c-grid" package="90136-1?04" value="90136-104" x="50" y="72"/>
+<element name="J1" library="con-molex-c-grid" package="90136-1?06" value="90136-106" x="15" y="72"/>
+<element name="J4" library="con-molex-c-grid" package="90136-1?08" value="90136-108" x="10" y="28" rot="R90"/>
+<element name="J5" library="con-molex-c-grid" package="90136-1?04" value="90136-104" x="10" y="51" rot="R270"/>
 </elements>
 <signals>
-<signal name="3V3">
-<contactref element="B1" pad="3V3"/>
-</signal>
 <signal name="5V">
 <contactref element="B1" pad="5V"/>
 </signal>
 <signal name="VCC">
-<contactref element="B1" pad="VIN"/>
 <contactref element="B2" pad="VIN"/>
 <contactref element="B3" pad="VCC"/>
 <contactref element="B4" pad="VCC"/>
-<contactref element="J1" pad="4"/>
 <contactref element="J2" pad="4"/>
-<wire x1="64.91" y1="29.24" x2="71.97" y2="49.27" width="0" layer="19" extent="1-1"/>
-<wire x1="64.73" y1="24.128" x2="64.91" y2="29.24" width="0" layer="19" extent="1-1"/>
+<contactref element="B1" pad="3V3"/>
+<contactref element="J1" pad="2"/>
+<contactref element="J4" pad="8"/>
+<contactref element="J5" pad="4"/>
+<wire x1="64.73" y1="24.128" x2="71.97" y2="49.27" width="0" layer="19" extent="1-1"/>
 <wire x1="46.02" y1="24.66" x2="64.73" y2="24.128" width="0" layer="19" extent="1-1"/>
-<wire x1="49.81" y1="72" x2="71.97" y2="49.27" width="0" layer="19" extent="1-1"/>
-<wire x1="32.81" y1="72" x2="49.81" y2="72" width="0" layer="19" extent="1-1"/>
+<wire x1="30.89" y1="29.24" x2="46.02" y2="24.66" width="0" layer="19" extent="1-1"/>
+<wire x1="10" y1="36.89" x2="30.89" y2="29.24" width="0" layer="19" extent="1-1"/>
+<wire x1="10" y1="47.19" x2="10" y2="36.89" width="0" layer="19" extent="1-1"/>
+<wire x1="11.19" y1="72" x2="10" y2="47.19" width="0" layer="19" extent="1-1"/>
+<wire x1="37.81" y1="72" x2="11.19" y2="72" width="0" layer="19" extent="1-1"/>
 </signal>
 <signal name="GND">
@@
 <contactref element="B3" pad="GND"/>
 <contactref element="B4" pad="GND"/>
-<contactref element="J1" pad="1"/>
 <contactref element="J2" pad="1"/>
 <contactref element="J2" pad="3"/>
+<contactref element="J1" pad="1"/>
+<contactref element="J1" pad="5"/>
+<contactref element="J1" pad="6"/>
+<contactref element="J4" pad="5"/>
+<contactref element="J5" pad="1"/>
 </signal>
 <signal name="IMU-SDA">
 <contactref element="B2" pad="SDA"/>
 <contactref element="B1" pad="D12"/>
-<wire x1="38.4" y1="24.66" x2="29.35" y2="44.48" width="0" layer="19" extent="1-1"/>
+<wire x1="38.4" y1="24.66" x2="28.35" y2="44.48" width="0" layer="19" extent="1-1"/>
 </signal>
 <signal name="IMU-SCL">
 <contactref element="B2" pad="SCL"/>
 <contactref element="B1" pad="A6"/>
-<wire x1="35.86" y1="24.66" x2="52.21" y2="29.24" width="0" layer="19" extent="1-1"/>
+<wire x1="35.86" y1="24.66" x2="51.21" y2="29.24" width="0" layer="19" extent="1-1"/>
 </signal>
 <signal name="GRN">
@@
 <contactref element="B3" pad="SDA"/>
 <contactref element="B1" pad="D4"/>
-<wire x1="49.67" y1="44.48" x2="59.27" y2="49.27" width="0" layer="19" extent="1-1"/>
+<wire x1="48.67" y1="44.48" x2="59.27" y2="49.27" width="0" layer="19" extent="1-1"/>
 </signal>
 <signal name="GPS-SCL">
 <contactref element="B3" pad="SCL"/>
 <contactref element="B1" pad="D5"/>
-<wire x1="47.13" y1="44.48" x2="61.81" y2="49.27" width="0" layer="19" extent="1-1"/>
+<wire x1="46.13" y1="44.48" x2="61.81" y2="49.27" width="0" layer="19" extent="1-1"/>
 </signal>
 <signal name="LOG-UART">
 <contactref element="B4" pad="RXI"/>
 <contactref element="B1" pad="A7"/>
-<wire x1="54.75" y1="29.24" x2="69.81" y2="24.128" width="0" layer="19" extent="1-1"/>
+<wire x1="53.75" y1="29.24" x2="69.81" y2="24.128" width="0" layer="19" extent="1-1"/>
 </signal>
 <signal name="CDH-TX">
 <contactref element="B1" pad="D1/TX"/>
-<contactref element="J1" pad="2"/>
-<wire x1="64.91" y1="44.48" x2="44.73" y2="72" width="0" layer="19" extent="1-1"/>
+<contactref element="J1" pad="3"/>
+<wire x1="13.73" y1="72" x2="63.91" y2="44.48" width="0" layer="19" extent="1-1"/>
 </signal>
 <signal name="CDH-RX">
 <contactref element="B1" pad="D0/RX"/>
-<contactref element="J1" pad="3"/>
-<wire x1="62.37" y1="44.48" x2="47.27" y2="72" width="0" layer="19" extent="1-1"/>
+<contactref element="J1" pad="4"/>
+<wire x1="16.27" y1="72" x2="61.37" y2="44.48" width="0" layer="19" extent="1-1"/>
 </signal>
 <signal name="SPI-MOSI">
 <contactref element="B1" pad="D2"/>
-</signal>
-<signal name="SPI-CS-ADC">
+<contactref element="J4" pad="7"/>
+<wire x1="10" y1="34.35" x2="53.75" y2="44.48" width="0" layer="19" extent="1-1"/>
+</signal>
+<signal name="SPI-CS-ADCS">
 <contactref element="B1" pad="D6"/>
+<contactref element="J4" pad="2"/>
+<wire x1="10" y1="21.65" x2="43.59" y2="44.48" width="0" layer="19" extent="1-1"/>
 </signal>
 <signal name="TEMP-OW">
 <contactref element="B1" pad="D9"/>
 <contactref element="J2" pad="2"/>
-<wire x1="36.97" y1="44.48" x2="27.73" y2="72" width="0" layer="19" extent="1-1"/>
+<wire x1="35.97" y1="44.48" x2="32.73" y2="72" width="0" layer="19" extent="1-1"/>
 </signal>
 <signal name="SPI-SCK">
 <contactref element="B1" pad="A1"/>
+<contactref element="J4" pad="4"/>
+<wire x1="10" y1="26.73" x2="38.51" y2="29.24" width="0" layer="19" extent="1-1"/>
 </signal>
 <signal name="SPI-MISO">
 <contactref element="B1" pad="A5"/>
+<contactref element="J4" pad="6"/>
+<wire x1="10" y1="31.81" x2="48.67" y2="29.24" width="0" layer="19" extent="1-1"/>
 </signal>
 <signal name="SPI-CS-ENV">
 <contactref element="B1" pad="D3"/>
-</signal>
-<signal name="N$1">
+<contactref element="J4" pad="1"/>
+<wire x1="10" y1="19.11" x2="51.21" y2="44.48" width="0" layer="19" extent="1-1"/>
+</signal>
+<signal name="DBG-RX">
+<contactref element="J3" pad="3"/>
+<contactref element="B1" pad="A2"/>
+<wire x1="41.05" y1="29.24" x2="51.27" y2="72" width="0" layer="19" extent="1-1"/>
+</signal>
+<signal name="DBG-TX">
+<contactref element="J3" pad="4"/>
+<contactref element="B1" pad="A0"/>
+<wire x1="35.97" y1="29.24" x2="53.81" y2="72" width="0" layer="19" extent="1-1"/>
+</signal>
+<signal name="VIN">
+<contactref element="B1" pad="VIN"/>
+</signal>
+<signal name="N$13">
+<contactref element="B1" pad="RST@2"/>
+</signal>
+<signal name="GPS-TX">
+<contactref element="B3" pad="TXD"/>
+<contactref element="J3" pad="2"/>
+<wire x1="64.35" y1="49.27" x2="48.73" y2="72" width="0" layer="19" extent="1-1"/>
+</signal>
+<signal name="GPS-RX">
+<contactref element="B3" pad="RXD"/>
 <contactref element="J3" pad="1"/>
-</signal>
-<signal name="N$2">
-<contactref element="J3" pad="2"/>
-</signal>
-<signal name="N$3">
-<contactref element="J3" pad="3"/>
-</signal>
-<signal name="N$4">
-<contactref element="J3" pad="4"/>
-</signal>
-<signal name="N$5">
-<contactref element="J4" pad="1"/>
-</signal>
-<signal name="N$6">
-<contactref element="J4" pad="2"/>
-</signal>
-<signal name="N$7">
+<wire x1="66.89" y1="49.27" x2="46.19" y2="72" width="0" layer="19" extent="1-1"/>
+</signal>
+<signal name="SPI-CS-SUN">
+<contactref element="B1" pad="D10"/>
 <contactref element="J4" pad="3"/>
-</signal>
-<signal name="N$8">
-<contactref element="J4" pad="4"/>
-</signal>
-<signal name="N$9">
-<contactref element="J4" pad="5"/>
-</signal>
-<signal name="N$10">
-<contactref element="J4" pad="6"/>
-</signal>
-<signal name="N$11">
-<contactref element="J4" pad="7"/>
-</signal>
-<signal name="N$12">
-<contactref element="J4" pad="8"/>
+<wire x1="10" y1="24.19" x2="33.43" y2="44.48" width="0" layer="19" extent="1-1"/>
+</signal>
+<signal name="SUN-RX">
+<contactref element="B1" pad="A4"/>
+<contactref element="J5" pad="2"/>
+<wire x1="10" y1="52.27" x2="46.13" y2="29.24" width="0" layer="19" extent="1-1"/>
+</signal>
+<signal name="SUN-TX">
+<contactref element="B1" pad="A3"/>
+<contactref element="J5" pad="3"/>
+<wire x1="10" y1="49.73" x2="43.59" y2="29.24" width="0" layer="19" extent="1-1"/>
 </signal>
 </signals>
