File: hardware/mainpanel/mainpanel.sch (EAGLE design)
At the start: 26 parts, among them J1 CDH, J2 OW, J3 DBG, J4 SUN-UART, J5 ADCS, J6 ENV, J7 SUN, U1 DS18B20, U2 DS18B20, U3 DS18B20

Commit message: Update lib
Parts:
- B1: device Frcy:NUCLEO-32 -> Frcy:NUCLEO-32BO
- B2: device Frcy:BOSCH-BNO055 -> Frcy:BOSCH-BNO055BO
- B3: device Frcy:UPUTRONICS-UBLOX-PICO -> Frcy:UPUTRONICS-UBLOX-PICOBO
- B4: device Frcy:SPARKFUN-OPENLOG -> Frcy:SPARKFUN-OPENLOGBO
Changed lines of the file:
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@@
 <setting verticaltext="up"/>
 </settings>
-<grid distance="0.1" unitdist="inch" unit="inch" style="lines" multiple="1" display="yes" altdistance="0.01" altunitdist="inch" altunit="inch"/>
+<grid distance="0.1" unitdist="inch" unit="inch" style="lines" multiple="1" display="no" altdistance="0.01" altunitdist="inch" altunit="inch"/>
 <layers>
 <layer number="1" name="Top" color="4" fill="1" visible="no" active="no"/>
@@
 </classes>
 <parts>
-<part name="B1" library="Frcy" deviceset="NUCLEO-32" device="" value="NUCLEO-32"/>
-<part name="B2" library="Frcy" deviceset="BOSCH-BNO055" device="" value="BNO055"/>
+<part name="B1" library="Frcy" deviceset="NUCLEO-32" device="BO" value="NUCLEO-32"/>
+<part name="B2" library="Frcy" deviceset="BOSCH-BNO055" device="BO" value="BNO055"/>
 <part name="P+1" library="supply1" library_urn="urn:adsk.eagle:library:371" deviceset="VCC" device=""/>
 <part name="GND1" library="supply1" library_urn="urn:adsk.eagle:library:371" deviceset="GND" device=""/>
-<part name="B3" library="Frcy" deviceset="UPUTRONICS-UBLOX-PICO" device="" value="UBLOX"/>
-<part name="B4" library="Frcy" deviceset="SPARKFUN-OPENLOG" device="" value="OPENLOG"/>
+<part name="B3" library="Frcy" deviceset="UPUTRONICS-UBLOX-PICO" device="BO" value="UBLOX"/>
+<part name="B4" library="Frcy" deviceset="SPARKFUN-OPENLOG" device="BO" value="OPENLOG"/>
 <part name="J2" library="con-molex-c-grid" deviceset="90136-1?04" device="" value="OW"/>
 <part name="J3" library="con-molex-c-grid" deviceset="90136-1?04" device="" value="DBG"/>
 <part name="J1" library="con-molex-c-grid" deviceset="90136-1?06" device="" value="CDH"/>
 <part name="R1" library="rcl" library_urn="urn:adsk.eagle:library:334" deviceset="R-EU_" device="R2012" package3d_urn="urn:adsk.eagle:package:23543/2" value="4.7k"/>
-<part name="U1" library="Frcy" deviceset="DS18B20" device=""/>
-<part name="U2" library="Frcy" deviceset="DS18B20" device=""/>
+<part name="U1" library="Frcy" deviceset="DS18B20" device="" value="DS18B20"/>
+<part name="U2" library="Frcy" deviceset="DS18B20" device="" value="DS18B20"/>
 <part name="R2" library="rcl" library_urn="urn:adsk.eagle:library:334" deviceset="R-EU_" device="R2012" package3d_urn="urn:adsk.eagle:package:23543/2" value="4.7k"/>
 <part name="J6" library="con-molex-c-grid" deviceset="90136-1?06" device="" value="ENV"/>
@@
 <part name="J7" library="con-molex-c-grid" deviceset="90136-1?06" device="" value="SUN"/>
 <part name="FRAME1" library="frames" library_urn="urn:adsk.eagle:library:229" deviceset="A4L-LOC" device=""/>
-<part name="U3" library="Frcy" deviceset="DS18B20" device=""/>
+<part name="U3" library="Frcy" deviceset="DS18B20" device="" value="DS18B20"/>
 <part name="R3" library="rcl" library_urn="urn:adsk.eagle:library:334" deviceset="R-EU_" device="R2012" package3d_urn="urn:adsk.eagle:package:23543/2" value="4.7k"/>
 <part name="R4" library="rcl" library_urn="urn:adsk.eagle:library:334" deviceset="R-EU_" device="R2012" package3d_urn="urn:adsk.eagle:package:23543/2" value="4.7k"/>

Commit message: Implement feedback
- BNO055 RST line
- Del BNO055 pullups
- 3 pin hdr for OW sensors
Parts:
- removed R3, R4: 4.7k, rcl:R-EU_R2012
- J2: device con-molex-c-grid:90136-104 -> con-molex-c-grid:90136-103
Connections:
- net N$1 renamed NUC-RST
- new net IMU-RST: B1.D11, B2.RST
- net GND: no longer J2.4
- net IMU-SCL: no longer R3.2
- net IMU-SDA: no longer R4.2
- net VCC: no longer R3.1, R4.1
Changed lines of the file:
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@@
 <setting verticaltext="up"/>
 </settings>
-<grid distance="0.1" unitdist="inch" unit="inch" style="lines" multiple="1" display="no" altdistance="0.01" altunitdist="inch" altunit="inch"/>
+<grid distance="0.1" unitdist="inch" unit="inch" style="lines" multiple="1" display="yes" altdistance="0.01" altunitdist="inch" altunit="inch"/>
 <layers>
 <layer number="1" name="Top" color="4" fill="1" visible="no" active="no"/>
@@
 <part name="B3" library="Frcy" deviceset="UPUTRONICS-UBLOX-PICO" device="BO" value="UBLOX"/>
 <part name="B4" library="Frcy" deviceset="SPARKFUN-OPENLOG" device="BO" value="OPENLOG"/>
-<part name="J2" library="con-molex-c-grid" deviceset="90136-1?04" device="" value="OW"/>
+<part name="J2" library="con-molex-c-grid" deviceset="90136-1?03" device="" value="OW"/>
 <part name="J3" library="con-molex-c-grid" deviceset="90136-1?04" device="" value="DBG"/>
 <part name="J1" library="con-molex-c-grid" deviceset="90136-1?06" device="" value="CDH"/>
@@
 <part name="FRAME1" library="frames" library_urn="urn:adsk.eagle:library:229" deviceset="A4L-LOC" device=""/>
 <part name="U3" library="Frcy" deviceset="DS18B20" device="" value="DS18B20"/>
-<part name="R3" library="rcl" library_urn="urn:adsk.eagle:library:334" deviceset="R-EU_" device="R2012" package3d_urn="urn:adsk.eagle:package:23543/2" value="4.7k"/>
-<part name="R4" library="rcl" library_urn="urn:adsk.eagle:library:334" deviceset="R-EU_" device="R2012" package3d_urn="urn:adsk.eagle:package:23543/2" value="4.7k"/>
 <part name="R5" library="rcl" library_urn="urn:adsk.eagle:library:334" deviceset="R-EU_" device="R2012" package3d_urn="urn:adsk.eagle:package:23543/2" value="4.7k"/>
 <part name="R6" library="rcl" library_urn="urn:adsk.eagle:library:334" deviceset="R-EU_" device="R2012" package3d_urn="urn:adsk.eagle:package:23543/2" value="4.7k"/>
@@
 </instance>
 <instance part="U3" gate="G$1" x="38.1" y="111.76"/>
-<instance part="R3" gate="G$1" x="195.58" y="142.24"/>
-<instance part="R4" gate="G$1" x="195.58" y="134.62"/>
 <instance part="R5" gate="G$1" x="195.58" y="111.76"/>
 <instance part="R6" gate="G$1" x="195.58" y="104.14"/>
@@
 <segment>
 <pinref part="B2" gate="G$1" pin="VIN"/>
-<wire x1="210.82" y1="160.02" x2="187.96" y2="160.02" width="0.1524" layer="91"/>
-<label x="185.42" y="160.02" size="1.27" layer="95" rot="R180" xref="yes"/>
-<wire x1="187.96" y1="160.02" x2="185.42" y2="160.02" width="0.1524" layer="91"/>
-<wire x1="187.96" y1="160.02" x2="187.96" y2="142.24" width="0.1524" layer="91"/>
-<junction x="187.96" y="160.02"/>
-<pinref part="R3" gate="G$1" pin="1"/>
-<wire x1="187.96" y1="142.24" x2="190.5" y2="142.24" width="0.1524" layer="91"/>
-<wire x1="187.96" y1="142.24" x2="187.96" y2="134.62" width="0.1524" layer="91"/>
-<junction x="187.96" y="142.24"/>
-<pinref part="R4" gate="G$1" pin="1"/>
-<wire x1="187.96" y1="134.62" x2="190.5" y2="134.62" width="0.1524" layer="91"/>
+<wire x1="210.82" y1="160.02" x2="200.66" y2="160.02" width="0.1524" layer="91"/>
+<label x="200.66" y="160.02" size="1.27" layer="95" rot="R180" xref="yes"/>
 </segment>
 <segment>
@@
 <junction x="109.22" y="27.94"/>
 </segment>
-<segment>
-<pinref part="J2" gate="G$1" pin="4"/>
-<wire x1="20.32" y1="48.26" x2="33.02" y2="48.26" width="0.1524" layer="91"/>
-<label x="33.02" y="48.26" size="1.27" layer="95" xref="yes"/>
-</segment>
 </net>
 <net name="IMU-SDA" class="0">
 <segment>
 <pinref part="B2" gate="G$1" pin="SDA"/>
-<wire x1="210.82" y1="152.4" x2="205.74" y2="152.4" width="0.1524" layer="91"/>
 <label x="200.66" y="152.4" size="1.27" layer="95" rot="R180" xref="yes"/>
-<pinref part="R4" gate="G$1" pin="2"/>
-<wire x1="205.74" y1="152.4" x2="200.66" y2="152.4" width="0.1524" layer="91"/>
-<wire x1="200.66" y1="134.62" x2="205.74" y2="134.62" width="0.1524" layer="91"/>
-<wire x1="205.74" y1="134.62" x2="205.74" y2="152.4" width="0.1524" layer="91"/>
-<junction x="205.74" y="152.4"/>
+<wire x1="210.82" y1="152.4" x2="200.66" y2="152.4" width="0.1524" layer="91"/>
 </segment>
 <segment>
@@
 <segment>
 <pinref part="B2" gate="G$1" pin="SCL"/>
-<wire x1="210.82" y1="149.86" x2="203.2" y2="149.86" width="0.1524" layer="91"/>
+<wire x1="210.82" y1="149.86" x2="200.66" y2="149.86" width="0.1524" layer="91"/>
 <label x="200.66" y="149.86" size="1.27" layer="95" rot="R180" xref="yes"/>
-<pinref part="R3" gate="G$1" pin="2"/>
-<wire x1="203.2" y1="149.86" x2="200.66" y2="149.86" width="0.1524" layer="91"/>
-<wire x1="200.66" y1="142.24" x2="203.2" y2="142.24" width="0.1524" layer="91"/>
-<wire x1="203.2" y1="142.24" x2="203.2" y2="149.86" width="0.1524" layer="91"/>
-<junction x="203.2" y="149.86"/>
 </segment>
 <segment>
@@
 </segment>
 </net>
-<net name="N$1" class="0">
+<net name="NUC-RST" class="0">
 <segment>
 <pinref part="B1" gate="G$1" pin="RST@2"/>
@@
 </segment>
 </net>
+<net name="IMU-RST" class="0">
+<segment>
+<pinref part="B1" gate="G$1" pin="D11"/>
+<wire x1="96.52" y1="101.6" x2="88.9" y2="101.6" width="0.1524" layer="91"/>
+<label x="88.9" y="101.6" size="1.27" layer="95" rot="R180" xref="yes"/>
+</segment>
+<segment>
+<pinref part="B2" gate="G$1" pin="RST"/>
+<wire x1="210.82" y1="147.32" x2="200.66" y2="147.32" width="0.1524" layer="91"/>
+<label x="200.66" y="147.32" size="1.27" layer="95" rot="R180" xref="yes"/>
+</segment>
+</net>

Commit message: Add BME680 onboard
Parts:
- added B5: BME680, Frcy:WATTEROT-BME680BO
Connections:
- new net ENO-CS: B1.D13, B5.7/CS
- net GND: now also B5.GND
- net SPI-MISO: now also B5.SDO/MISO
- net SPI-MOSI: now also B5.SDA/MOSI
- net SPI-SCK: now also B5.SCL/SCK
- net VCC: now also B5.VCC
Other:
- moved on the sheet: B2, B3, B4, R5, R6

Commit message: Move components
Parts:
- C1: value 0.1uF -> 0.2uF
Connections:
- net ENO-CS renamed SPI-CS-ENO
- net DBG-RX: now also B1.A4; no longer B1.A2
- net DBG-TX: now also B1.A3; no longer B1.A0
- net GND: now also J5.4, J6.4, J7.4; no longer J5.3, J6.3, J7.3
- net SPI-MISO: now also J5.2, J6.2, J7.2; no longer J5.4, J6.4, J7.4
- net SPI-MOSI: now also J5.3, J6.3, J7.3; no longer J5.5, J6.5, J7.5
- net SPI-SCK: now also J5.5, J6.5, J7.5; no longer J5.2, J6.2, J7.2
- net SUN-RX: now also B1.A2; no longer B1.A4
- net SUN-TX: now also B1.A0; no longer B1.A3
- net TEMP-OW: now also R1.2; no longer R1.1
- net VCC: now also R1.1; no longer R1.2

Commit message: Add power connections
Connections:
- net TEMP-OW: now also R1.1; no longer R1.2
- net VCC: now also R1.2; no longer R1.1
Changed lines of the file:
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@@
 <pinref part="U1" gate="G$1" pin="VDD"/>
 <wire x1="27.94" y1="162.56" x2="25.4" y2="162.56" width="0.1524" layer="91"/>
-<wire x1="25.4" y1="162.56" x2="25.4" y2="139.7" width="0.1524" layer="91"/>
+<wire x1="25.4" y1="162.56" x2="25.4" y2="147.32" width="0.1524" layer="91"/>
 <pinref part="U2" gate="G$1" pin="VDD"/>
+<wire x1="25.4" y1="147.32" x2="25.4" y2="139.7" width="0.1524" layer="91"/>
 <wire x1="25.4" y1="139.7" x2="27.94" y2="139.7" width="0.1524" layer="91"/>
 <label x="25.4" y="162.56" size="1.27" layer="95" rot="R180" xref="yes"/>
-<wire x1="25.4" y1="139.7" x2="25.4" y2="132.08" width="0.1524" layer="91"/>
 <junction x="25.4" y="139.7"/>
 <pinref part="U3" gate="G$1" pin="VDD"/>
-<wire x1="25.4" y1="132.08" x2="25.4" y2="116.84" width="0.1524" layer="91"/>
+<wire x1="25.4" y1="139.7" x2="25.4" y2="116.84" width="0.1524" layer="91"/>
 <wire x1="25.4" y1="116.84" x2="27.94" y2="116.84" width="0.1524" layer="91"/>
-<pinref part="R1" gate="G$1" pin="1"/>
-<wire x1="12.7" y1="134.62" x2="12.7" y2="132.08" width="0.1524" layer="91"/>
-<wire x1="12.7" y1="132.08" x2="25.4" y2="132.08" width="0.1524" layer="91"/>
-<junction x="25.4" y="132.08"/>
+<pinref part="R1" gate="G$1" pin="2"/>
+<wire x1="12.7" y1="144.78" x2="12.7" y2="147.32" width="0.1524" layer="91"/>
+<wire x1="12.7" y1="147.32" x2="25.4" y2="147.32" width="0.1524" layer="91"/>
+<junction x="25.4" y="147.32"/>
 </segment>
 <segment>
@@
 <wire x1="27.94" y1="157.48" x2="22.86" y2="157.48" width="0.1524" layer="91"/>
 <pinref part="U2" gate="G$1" pin="DQ"/>
-<wire x1="22.86" y1="157.48" x2="22.86" y2="147.32" width="0.1524" layer="91"/>
-<wire x1="22.86" y1="147.32" x2="22.86" y2="134.62" width="0.1524" layer="91"/>
+<wire x1="22.86" y1="157.48" x2="22.86" y2="134.62" width="0.1524" layer="91"/>
 <wire x1="22.86" y1="134.62" x2="27.94" y2="134.62" width="0.1524" layer="91"/>
 <label x="22.86" y="157.48" size="1.27" layer="95" rot="R180" xref="yes"/>
 <junction x="22.86" y="134.62"/>
-<wire x1="22.86" y1="134.62" x2="22.86" y2="111.76" width="0.1524" layer="91"/>
+<wire x1="22.86" y1="134.62" x2="22.86" y2="132.08" width="0.1524" layer="91"/>
 <pinref part="U3" gate="G$1" pin="DQ"/>
+<wire x1="22.86" y1="132.08" x2="22.86" y2="111.76" width="0.1524" layer="91"/>
 <wire x1="22.86" y1="111.76" x2="27.94" y2="111.76" width="0.1524" layer="91"/>
-<pinref part="R1" gate="G$1" pin="2"/>
-<wire x1="12.7" y1="144.78" x2="12.7" y2="147.32" width="0.1524" layer="91"/>
-<wire x1="12.7" y1="147.32" x2="22.86" y2="147.32" width="0.1524" layer="91"/>
-<junction x="22.86" y="147.32"/>
-</segment>
-<segment>
+<pinref part="R1" gate="G$1" pin="1"/>
+<wire x1="12.7" y1="134.62" x2="12.7" y2="132.08" width="0.1524" layer="91"/>
+<wire x1="12.7" y1="132.08" x2="22.86" y2="132.08" width="0.1524" layer="91"/>
+<junction x="22.86" y="132.08"/>
+</segment>
+<segment>

Commit message: Update spi connectors
Connections:
- net GND: now also J5.5, J6.5, J7.5; no longer J5.4, J6.4, J7.4
- net SPI-SCK: now also J5.4, J6.4, J7.4; no longer J5.5, J6.5, J7.5
Changed lines of the file:
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@@
 </segment>
 <segment>
-<wire x1="106.68" y1="25.4" x2="109.22" y2="25.4" width="0.1524" layer="91"/>
-<label x="119.38" y="25.4" size="1.27" layer="95" xref="yes"/>
-<pinref part="J7" gate="G$1" pin="4"/>
+<wire x1="20.32" y1="22.86" x2="22.86" y2="22.86" width="0.1524" layer="91"/>
+<label x="33.02" y="22.86" size="1.27" layer="95" xref="yes"/>
+<pinref part="J5" gate="G$1" pin="5"/>
+<pinref part="C5" gate="G$1" pin="1"/>
+<wire x1="22.86" y1="22.86" x2="33.02" y2="22.86" width="0.1524" layer="91"/>
+<wire x1="22.86" y1="10.16" x2="22.86" y2="22.86" width="0.1524" layer="91"/>
+<junction x="22.86" y="22.86"/>
+</segment>
+<segment>
+<wire x1="63.5" y1="22.86" x2="66.04" y2="22.86" width="0.1524" layer="91"/>
+<label x="76.2" y="22.86" size="1.27" layer="95" xref="yes"/>
+<pinref part="J6" gate="G$1" pin="5"/>
+<pinref part="C6" gate="G$1" pin="1"/>
+<wire x1="66.04" y1="22.86" x2="76.2" y2="22.86" width="0.1524" layer="91"/>
+<wire x1="66.04" y1="10.16" x2="66.04" y2="22.86" width="0.1524" layer="91"/>
+<junction x="66.04" y="22.86"/>
+</segment>
+<segment>
+<wire x1="106.68" y1="22.86" x2="109.22" y2="22.86" width="0.1524" layer="91"/>
+<label x="119.38" y="22.86" size="1.27" layer="95" xref="yes"/>
+<pinref part="J7" gate="G$1" pin="5"/>
 <pinref part="C7" gate="G$1" pin="1"/>
-<wire x1="109.22" y1="25.4" x2="119.38" y2="25.4" width="0.1524" layer="91"/>
-<wire x1="109.22" y1="10.16" x2="109.22" y2="25.4" width="0.1524" layer="91"/>
-<junction x="109.22" y="25.4"/>
-</segment>
-<segment>
-<wire x1="63.5" y1="25.4" x2="66.04" y2="25.4" width="0.1524" layer="91"/>
-<label x="76.2" y="25.4" size="1.27" layer="95" xref="yes"/>
-<pinref part="J6" gate="G$1" pin="4"/>
-<pinref part="C6" gate="G$1" pin="1"/>
-<wire x1="66.04" y1="25.4" x2="76.2" y2="25.4" width="0.1524" layer="91"/>
-<wire x1="66.04" y1="10.16" x2="66.04" y2="25.4" width="0.1524" layer="91"/>
-<junction x="66.04" y="25.4"/>
-</segment>
-<segment>
-<wire x1="20.32" y1="25.4" x2="22.86" y2="25.4" width="0.1524" layer="91"/>
-<label x="33.02" y="25.4" size="1.27" layer="95" xref="yes"/>
-<pinref part="J5" gate="G$1" pin="4"/>
-<pinref part="C5" gate="G$1" pin="1"/>
-<wire x1="22.86" y1="25.4" x2="33.02" y2="25.4" width="0.1524" layer="91"/>
-<wire x1="22.86" y1="10.16" x2="22.86" y2="25.4" width="0.1524" layer="91"/>
-<junction x="22.86" y="25.4"/>
+<wire x1="109.22" y1="22.86" x2="119.38" y2="22.86" width="0.1524" layer="91"/>
+<wire x1="109.22" y1="10.16" x2="109.22" y2="22.86" width="0.1524" layer="91"/>
+<junction x="109.22" y="22.86"/>
 </segment>
 </net>
@@
 </segment>
 <segment>
-<wire x1="20.32" y1="22.86" x2="33.02" y2="22.86" width="0.1524" layer="91"/>
-<label x="33.02" y="22.86" size="1.27" layer="95" xref="yes"/>
-<pinref part="J5" gate="G$1" pin="5"/>
-</segment>
-<segment>
-<wire x1="63.5" y1="22.86" x2="76.2" y2="22.86" width="0.1524" layer="91"/>
-<label x="76.2" y="22.86" size="1.27" layer="95" xref="yes"/>
-<pinref part="J6" gate="G$1" pin="5"/>
-</segment>
-<segment>
-<wire x1="106.68" y1="22.86" x2="119.38" y2="22.86" width="0.1524" layer="91"/>
-<label x="119.38" y="22.86" size="1.27" layer="95" xref="yes"/>
-<pinref part="J7" gate="G$1" pin="5"/>
-</segment>
-</net>
+<label x="33.02" y="25.4" size="1.27" layer="95" xref="yes"/>
+<pinref part="J5" gate="G$1" pin="4"/>
+<wire x1="20.32" y1="25.4" x2="33.02" y2="25.4" width="0.1524" layer="91"/>
+</segment>
+<segment>
+<label x="76.2" y="25.4" size="1.27" layer="95" xref="yes"/>
+<pinref part="J6" gate="G$1" pin="4"/>
+<wire x1="63.5" y1="25.4" x2="76.2" y2="25.4" width="0.1524" layer="91"/>
+</segment>
+<segment>
+<label x="119.38" y="25.4" size="1.27" layer="95" xref="yes"/>
+<pinref part="J7" gate="G$1" pin="4"/>
+<wire x1="106.68" y1="25.4" x2="119.38" y2="25.4" width="0.1524" layer="91"/>
+</segment>
+</net>

Commit message: Improve layout
Connections:
- net GND: now also C2.2; no longer C2.1
- net VCC: now also C2.1; no longer C2.2
Changed lines of the file:
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@@
 <segment>
 <pinref part="J2" gate="G$1" pin="3"/>
-<wire x1="20.32" y1="50.8" x2="30.48" y2="50.8" width="0.1524" layer="91"/>
+<wire x1="20.32" y1="50.8" x2="22.86" y2="50.8" width="0.1524" layer="91"/>
 <label x="33.02" y="50.8" size="1.27" layer="95" xref="yes"/>
-<pinref part="C2" gate="G$1" pin="2"/>
-<wire x1="30.48" y1="50.8" x2="33.02" y2="50.8" width="0.1524" layer="91"/>
-<wire x1="30.48" y1="58.42" x2="30.48" y2="50.8" width="0.1524" layer="91"/>
-<junction x="30.48" y="50.8"/>
+<pinref part="C2" gate="G$1" pin="1"/>
+<wire x1="22.86" y1="50.8" x2="33.02" y2="50.8" width="0.1524" layer="91"/>
+<wire x1="22.86" y1="58.42" x2="22.86" y2="50.8" width="0.1524" layer="91"/>
+<junction x="22.86" y="50.8"/>
 </segment>
 <segment>
@@
 <segment>
 <pinref part="J2" gate="G$1" pin="1"/>
-<wire x1="20.32" y1="55.88" x2="22.86" y2="55.88" width="0.1524" layer="91"/>
 <label x="33.02" y="55.88" size="1.27" layer="95" xref="yes"/>
-<pinref part="C2" gate="G$1" pin="1"/>
-<wire x1="22.86" y1="55.88" x2="33.02" y2="55.88" width="0.1524" layer="91"/>
-<wire x1="22.86" y1="58.42" x2="22.86" y2="55.88" width="0.1524" layer="91"/>
-<junction x="22.86" y="55.88"/>
+<wire x1="20.32" y1="55.88" x2="30.48" y2="55.88" width="0.1524" layer="91"/>
+<pinref part="C2" gate="G$1" pin="2"/>
+<wire x1="30.48" y1="55.88" x2="33.02" y2="55.88" width="0.1524" layer="91"/>
+<wire x1="30.48" y1="58.42" x2="30.48" y2="55.88" width="0.1524" layer="91"/>
+<junction x="30.48" y="55.88"/>
 </segment>
 <segment>
@@
 <label x="22.86" y="157.48" size="1.27" layer="95" rot="R180" xref="yes"/>
 <junction x="22.86" y="134.62"/>
+<pinref part="U3" gate="G$1" pin="DQ"/>
 <wire x1="22.86" y1="134.62" x2="22.86" y2="132.08" width="0.1524" layer="91"/>
-<pinref part="U3" gate="G$1" pin="DQ"/>
 <wire x1="22.86" y1="132.08" x2="22.86" y2="111.76" width="0.1524" layer="91"/>
 <wire x1="22.86" y1="111.76" x2="27.94" y2="111.76" width="0.1524" layer="91"/>
