File: hardware/sensors.brd (EAGLE design)
At the start: 80 x 80 mm, 31 parts, among them U1 DS18B20, U2 DS18B20, U3 DS18B20

Commit message: Reroute I2C connections
Parts:
- moved R5 26.1 mm to (62.0, 62.0), turned to 270 degrees
- moved R6 23.0 mm to (59.0, 62.0), turned to 270 degrees
Routing:
- net GPS-SDA: track 47.6 -> 31.4 mm
- net GPS-SCL: track 53.7 -> 37.7 mm, vias 0 -> 2
- net VCC: track 87.0 -> 90.2 mm, vias 19 -> 20
- net GPS-TP: track 69.3 -> 70.7 mm
- net CDH-RX: track 42.6 -> 43.3 mm
- net CDH-TX: track 42.3 -> 43.0 mm
